Commit message: Update latest changes

File: description/robot.urdf.xacro (robot description, xacro)
@@ -1,5 +1,7 @@
 <?xml version="1.0"?>
 <robot xmlns:xacro="http://www.ros.org/wiki/xacro"  name="robot">
-    <!-- Example link -->
+    <!-- basic describe: 3 wheels, 1 CHASSIS -->
     <xacro:include filename="robot_core.xacro" />
+    <!-- Control 2 wheel: left & right-->
+    <xacro:include filename="robot_control.xacro" />
 </robot>

File: description/robot_core.xacro (robot description, xacro)
@@ -45,4 +45,9 @@
         </xacro:inertial_box>
     </link>
+    <gazebo reference="chassis">
+        <material>
+            Gazebo/White
+        </material>
+    </gazebo>
     <!-- LEFT WHEEL LINK -->
     <joint name="left_wheel_joint" type="continuous">
@@ -69,4 +74,9 @@
         </xacro:inertial_cylinder>
     </link>
+    <gazebo reference="left_wheel">
+        <material>
+            Gazebo/Blue
+        </material>
+    </gazebo>
         <!-- RIGHT WHEEL LINK -->
     <joint name="right_wheel_joint" type="continuous">
@@ -93,4 +103,9 @@
         </xacro:inertial_cylinder>
     </link>
+    <gazebo reference="right_wheel">
+        <material>
+            Gazebo/Blue
+        </material>
+    </gazebo>
     <!-- CASTER WHEEL LINK-->
     <joint name="caster_wheel_joint" type="fixed">
@@ -116,3 +131,11 @@
         </xacro:inertial_sphere>
     </link>
+    <gazebo reference="caster_wheel">
+        <material>
+            Gazebo/Black
+        </material>
+        <!-- hệ số ma sát cho ( x,y), nếu không setup thì caster wheel bị khóa cứng -> xe nhảy tưng tưng-->
+        <mu1 value="0.001"/>
+        <mu2 value="0.001"/>
+    </gazebo>
 </robot>

Commit message: update

File: description/robot.urdf.xacro (robot description, xacro)
@@ -5,3 +5,6 @@
     <!-- Control 2 wheel: left & right-->
     <xacro:include filename="robot_control.xacro" />
+    <!-- Control lidar-->
+    <xacro:include filename="lidar.xacro" />
+    <xacro:include filename="camera.xacro" />
 </robot>

File: description/robot_core.xacro (robot description, xacro)
@@ -13,4 +13,7 @@
     <material name="black">
         <color rgba="0 0 0 1"/>
+    </material>
+    <material name="red">
+    <color rgba="1 0 0 1"/>
     </material>
     <!-- BASE LINK-->
